File: Hardware/Balance PCB/robot_balance.brd (EAGLE design)
At the start: 100 x 50 mm, 50 parts, among them P1 10118194-0001LF, Q1 16Mhz

Commit message: updates
Parts:
- moved R_EN 77.7 mm to (62.0, 38.0), turned to 90 degrees
- flipped C1 to the top
- flipped C2 to the top
Changed lines of the file:
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@@
 <element name="3.3_PWR" library="LilyPad-Wearables" package="LED-1206" value="" x="41" y="18"/>
 <element name="BATT_PWR" library="LilyPad-Wearables" package="LED-1206" value="" x="41" y="32"/>
-<element name="C1" library="SparkFun-Capacitors" package="0805" value="2.2uF" x="75" y="21" rot="MR90">
-<attribute name="PROD_ID" value="CAP-11624" x="75" y="21" size="1.778" layer="28" rot="MR90" display="off"/>
+<element name="C1" library="SparkFun-Capacitors" package="0805" value="2.2uF" x="75" y="21" rot="R90">
+<attribute name="PROD_ID" value="CAP-11624" x="75" y="21" size="1.778" layer="27" rot="R90" display="off"/>
 </element>
 <element name="C12" library="SparkFun-Capacitors" package="0805" value="0.1uF" x="66" y="16" rot="R270">
@@
 <element name="C16" library="SparkFun-Capacitors" package="0805" value="12pF" x="53" y="21" rot="R270"/>
 <element name="C17" library="SparkFun-Capacitors" package="0805" value="12pF" x="53" y="31" rot="R90"/>
-<element name="C2" library="SparkFun-Capacitors" package="0805" value="2.2uF" x="77" y="21" rot="MR90">
-<attribute name="PROD_ID" value="CAP-11624" x="77" y="21" size="1.778" layer="28" rot="MR90" display="off"/>
+<element name="C2" library="SparkFun-Capacitors" package="0805" value="2.2uF" x="77" y="21" rot="R90">
+<attribute name="PROD_ID" value="CAP-11624" x="77" y="21" size="1.778" layer="27" rot="R90" display="off"/>
 </element>
 <element name="C24" library="SparkFun-Capacitors" package="0805" value="0.1uF" x="76" y="29">
@@
 </element>
 <element name="JP3" library="SparkFun-Connectors" package="MOLEX-1X6_LOCK" value="" x="62" y="43"/>
-<element name="R_EN" library="SparkFun-Passives" package="0603-RES" value="1K" x="-2" y="-6"/>
+<element name="R_EN" library="SparkFun-Passives" package="0603-RES" value="1K" x="62" y="38" rot="R90"/>
 </elements>
 <signals>
@@
 <contactref element="JP3" pad="4"/>
 <contactref element="P1" pad="5"/>
-<wire x1="86.81" y1="41" x2="94.97" y2="34.19" width="0" layer="19" extent="1-1"/>
-<wire x1="94.97" y1="18.95" x2="94.97" y2="34.19" width="0" layer="19" extent="1-1"/>
-<wire x1="76.9" y1="29" x2="86.81" y2="41" width="0" layer="19" extent="1-1"/>
-<wire x1="76.9" y1="26" x2="76.9" y2="29" width="0" layer="19" extent="1-1"/>
-<wire x1="72" y1="35.9" x2="76.9" y2="29" width="0" layer="19" extent="1-1"/>
-<wire x1="69.62" y1="42.746" x2="72" y2="35.9" width="0" layer="19" extent="1-1"/>
-<wire x1="63" y1="35.9" x2="72" y2="35.9" width="0" layer="19" extent="1-1"/>
-<wire x1="62.75" y1="30.8" x2="63" y2="35.9" width="0" layer="19" extent="1-1"/>
-<wire x1="60.15" y1="23.25" x2="62.75" y2="30.8" width="0" layer="19" extent="1-1"/>
-<wire x1="62.75" y1="19.2" x2="60.15" y2="23.25" width="0" layer="19" extent="1-1"/>
-<wire x1="63" y1="15.1" x2="62.75" y2="19.2" width="0" layer="19" extent="1-1"/>
-<wire x1="66" y1="15.1" x2="63" y2="15.1" width="0" layer="19" extent="1-1"/>
-<wire x1="70" y1="15.1" x2="66" y2="15.1" width="0" layer="19" extent="1-1"/>
-<wire x1="73" y1="15.1" x2="70" y2="15.1" width="0" layer="19" extent="1-1"/>
-<wire x1="61.89" y1="10.27" x2="63" y2="15.1" width="0" layer="19" extent="1-1"/>
-<wire x1="64.43" y1="10.27" x2="61.89" y2="10.27" width="0" layer="19" extent="1-1"/>
-<wire x1="59.35" y1="10.27" x2="61.89" y2="10.27" width="0" layer="19" extent="1-1"/>
-<wire x1="56.81" y1="10.27" x2="59.35" y2="10.27" width="0" layer="19" extent="1-1"/>
-<wire x1="54.27" y1="10.27" x2="56.81" y2="10.27" width="0" layer="19" extent="1-1"/>
-<wire x1="51.73" y1="10.27" x2="54.27" y2="10.27" width="0" layer="19" extent="1-1"/>
-<wire x1="49.19" y1="10.27" x2="51.73" y2="10.27" width="0" layer="19" extent="1-1"/>
-<wire x1="46.65" y1="10.27" x2="49.19" y2="10.27" width="0" layer="19" extent="1-1"/>
-<wire x1="44.11" y1="10.27" x2="46.65" y2="10.27" width="0" layer="19" extent="1-1"/>
-<wire x1="55.1" y1="18" x2="60.15" y2="23.25" width="0" layer="19" extent="1-1"/>
-<wire x1="53" y1="20.1" x2="55.1" y2="18" width="0" layer="19" extent="1-1"/>
-<wire x1="52.2" y1="24.9" x2="53" y2="20.1" width="0" layer="19" extent="1-1"/>
-<wire x1="53.8" y1="27.1" x2="52.2" y2="24.9" width="0" layer="19" extent="1-1"/>
-<wire x1="53" y1="31.9" x2="53.8" y2="27.1" width="0" layer="19" extent="1-1"/>
-<wire x1="47.9" y1="32" x2="53" y2="31.9" width="0" layer="19" extent="1-1"/>
-<wire x1="47.9" y1="18" x2="53" y2="20.1" width="0" layer="19" extent="1-1"/>
-<wire x1="48" y1="40.1" x2="47.9" y2="32" width="0" layer="19" extent="1-1"/>
-<wire x1="52" y1="40.1" x2="48" y2="40.1" width="0" layer="19" extent="1-1"/>
-<wire x1="44" y1="40.1" x2="48" y2="40.1" width="0" layer="19" extent="1-1"/>
-<wire x1="40" y1="40.1" x2="44" y2="40.1" width="0" layer="19" extent="1-1"/>
-<wire x1="33.5" y1="44.3" x2="40" y2="40.1" width="0" layer="19" extent="1-1"/>
-<wire x1="34.5" y1="47" x2="33.5" y2="44.3" width="0" layer="19" extent="1-1"/>
-<wire x1="29.7" y1="44.3" x2="33.5" y2="44.3" width="0" layer="19" extent="1-1"/>
-<wire x1="28.5" y1="44.3" x2="29.7" y2="44.3" width="0" layer="19" extent="1-1"/>
-<wire x1="27.5" y1="47" x2="28.5" y2="44.3" width="0" layer="19" extent="1-1"/>
-<wire x1="41.9012" y1="26" x2="47.9" y2="32" width="0" layer="19" extent="1-1"/>
-<wire x1="38" y1="27.1" x2="41.9012" y2="26" width="0" layer="19" extent="1-1"/>
-<wire x1="38" y1="24.9" x2="38" y2="27.1" width="0" layer="19" extent="1-1"/>
-<wire x1="33.656" y1="30.675" x2="38" y2="27.1" width="0" layer="19" extent="1-1"/>
-<wire x1="26.344" y1="31.325" x2="33.656" y2="30.675" width="0" layer="19" extent="1-1"/>
-<wire x1="26.344" y1="33.275" x2="26.344" y2="31.325" width="0" layer="19" extent="1-1"/>
-<wire x1="26.344" y1="28.725" x2="26.344" y2="31.325" width="0" layer="19" extent="1-1"/>
-<wire x1="26.344" y1="28.075" x2="26.344" y2="28.725" width="0" layer="19" extent="1-1"/>
-<wire x1="23" y1="32.15" x2="26.344" y2="31.325" width="0" layer="19" extent="1-1"/>
-<wire x1="17.97" y1="34.19" x2="23" y2="32.15" width="0" layer="19" extent="1-1"/>
-<wire x1="24.206" y1="19.905" x2="26.344" y2="28.075" width="0" layer="19" extent="1-1"/>
-<wire x1="29.794" y1="19.905" x2="24.206" y2="19.905" width="0" layer="19" extent="1-1"/>
-<wire x1="34.9" y1="17" x2="29.794" y2="19.905" width="0" layer="19" extent="1-1"/>
-<wire x1="17.97" y1="18.95" x2="24.206" y2="19.905" width="0" layer="19" extent="1-1"/>
-<wire x1="10.35" y1="41" x2="17.97" y2="34.19" width="0" layer="19" extent="1-1"/>
-<wire x1="79.62" y1="5.873" x2="73" y2="15.1" width="0" layer="19" extent="1-1"/>
 </signal>
 <signal name="3.3V" class="3">
@@
 <contactref element="C1" pad="1"/>
 <contactref element="U$4" pad="31"/>
-<wire x1="75" y1="20.1" x2="77" y2="20.1" width="0" layer="19" extent="16-16"/>
-<wire x1="69.25" y1="19.2" x2="75" y2="20.1" width="0" layer="19" extent="1-16"/>
+<wire x1="75" y1="20.1" x2="77" y2="20.1" width="0" layer="19" extent="1-1"/>
+<wire x1="69.25" y1="19.2" x2="75" y2="20.1" width="0" layer="19" extent="1-1"/>
 </signal>
 <signal name="N$12">
@@
 <contactref element="C2" pad="2"/>
 <contactref element="U$4" pad="47"/>
-<wire x1="75" y1="21.9" x2="71.85" y2="28.25" width="0" layer="19" extent="1-16"/>
-<wire x1="77" y1="21.9" x2="75" y2="21.9" width="0" layer="19" extent="16-16"/>
+<wire x1="75" y1="21.9" x2="71.85" y2="28.25" width="0" layer="19" extent="1-1"/>
+<wire x1="77" y1="21.9" x2="75" y2="21.9" width="0" layer="19" extent="1-1"/>
 </signal>
 <signal name="N$41" class="1">
@@
 <contactref element="JP3" pad="1"/>
 <contactref element="R_EN" pad="1"/>
-<wire x1="-2.85" y1="-6" x2="62" y2="43" width="0" layer="19" extent="1-1"/>
+<wire x1="62" y1="37.15" x2="62" y2="43" width="0" layer="19" extent="1-1"/>
 </signal>
 <signal name="N$6">
 <contactref element="U$4" pad="40"/>
 <contactref element="R_EN" pad="2"/>
-<wire x1="-1.15" y1="-6" x2="71.85" y2="24.75" width="0" layer="19" extent="1-1"/>
+<wire x1="71.85" y1="24.75" x2="62" y2="38.85" width="0" layer="19" extent="1-1"/>
 </signal>
 </signals>

Commit message: Added VCP solder jumpers
Parts:
- added JP4, JP6: (no value), SparkFun-Retired:SJ_2S-NO
Connections:
- new net USB_DM: JP4.1, U$4.44
- new net USB_DP: JP6.1, U$4.45
- net USB_D+: now also JP6.2
- net USB_D-: now also JP4.2
Changed lines of the file:
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@@
 <element name="JP3" library="SparkFun-Connectors" package="MOLEX-1X6_LOCK" value="" x="62" y="43"/>
 <element name="R_EN" library="SparkFun-Passives" package="0603-RES" value="1K" x="62" y="38" rot="R90"/>
+<element name="JP4" library="SparkFun-Retired" package="SJ_2S-NO" value="" x="36" y="41" rot="R180"/>
+<element name="JP6" library="SparkFun-Retired" package="SJ_2S-NO" value="" x="36" y="38" rot="R180"/>
 </elements>
 <signals>
@@
 <contactref element="FT232RL" pad="16"/>
 <contactref element="P1" pad="2"/>
+<contactref element="JP4" pad="2"/>
+<wire x1="35.55" y1="41" x2="31.65" y2="44.3" width="0" layer="19" extent="1-1"/>
 <wire x1="26.344" y1="34.575" x2="31.65" y2="44.3" width="0" layer="19" extent="1-1"/>
 </signal>
@@
 <contactref element="FT232RL" pad="15"/>
 <contactref element="P1" pad="3"/>
-<wire x1="26.344" y1="35.225" x2="31" y2="44.3" width="0" layer="19" extent="1-1"/>
+<contactref element="JP6" pad="2"/>
+<wire x1="35.55" y1="38" x2="31" y2="44.3" width="0" layer="19" extent="1-1"/>
+<wire x1="26.344" y1="35.225" x2="35.55" y2="38" width="0" layer="19" extent="1-1"/>
 </signal>
 <signal name="5V" class="3">
@@
 <wire x1="71.85" y1="24.75" x2="62" y2="38.85" width="0" layer="19" extent="1-1"/>
 </signal>
+<signal name="USB_DM">
+<contactref element="JP4" pad="1"/>
+<contactref element="U$4" pad="44"/>
+<wire x1="36.45" y1="41" x2="71.85" y2="26.75" width="0" layer="19" extent="1-1"/>
+</signal>
+<signal name="USB_DP">
+<contactref element="JP6" pad="1"/>
+<contactref element="U$4" pad="45"/>
+<wire x1="36.45" y1="38" x2="71.85" y2="27.25" width="0" layer="19" extent="1-1"/>
+</signal>
 </signals>
